File: ESP32-2-Relay.kicad_sch (KiCad schematic)
At the start: 44 parts, among them J1 Relay-1, J2 Relay-2, J3 USB_C_Receptacle_USB2.0, K1 SRD-05VDC-SL-C, K2 SRD-05VDC-SL-C, Q1 BC857, Q2 BC857, Q3 BC847W, Q4 BC847W, SW3 SW_Push, SW4 SW_Push, U1 AMS1117-3.3, U4 ESP32-WROOM-32, U5 PC817, U6 PC817, U7 USBLC6-2SC6, U8 CP2102N-Axx-xQFN28

Commit message: 17h
Parts:
- R1: footprint Resistor_SMD:R_0402_1005Metric -> Resistor_SMD:R_0603_1608Metric
Connections:
- net +3.3V is gone; now on net +3V3: C2.1, U1.2 (VO)
- net DTR: now also U8.1 (~{DCD}); no longer U8.28 (~{DTR})
- net IO_34: now reaches U4.6 (IO34)
- net IO_34: now also D2.1 (K)
- net IO_35: now reaches U4.7 (IO35)
- net IO_35: now also D4.1 (K)
- net IO_19: no longer names the net of U4.31 (IO19)
- net IO_19: no longer D4.1 (K)
- net IO_21: no longer names the net of U4.33 (IO21)
- net IO_21: no longer D2.1 (K)
Other:
- note added: "5V to 3.3V"
- note added: "Button"
- note added: "CP2102"
- note removed: "Voltage Regulator 5V to 3.3V"
- moved on the sheet: C10, C3, C4, D2, D3, D4, D5, D8, J1, J2, J3, K1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

Commit message: done
Parts:
- removed C1: 22uF, Capacitor_SMD:C_0201_0603Metric, symbol Device:C_Small
- added J4: Conn_01x02, TRUNGTHAO:Conn_XH-P2.54mm-2P, symbol TrungThao7112024:Conn_01x02
Connections:
- net +5V: now also J4.2 (Pin_2)
- net GND: now also J4.1 (Pin_1)
